File: TeslaCoil.kicad_pcb (KiCad board)
At the start: 2 copper layers, 100 x 101 mm, 0 parts

Commit message: layout mockup
Parts:
- added C1: 20uF, Capacitor_THT:CP_Radial_D17.0mm_P7.50mm, F.Cu at (82.5, 88.5)
- added C12: 0.1u, Capacitor_SMD:C_0805_2012Metric_Pad1.18x1.45mm_HandSolder, F.Cu at (158.0, 122.0)
- added C13: 1u, Capacitor_SMD:C_0805_2012Metric_Pad1.18x1.45mm_HandSolder, F.Cu at (158.0, 125.0)
- added C14: 20uF, Capacitor_SMD:C_0805_2012Metric_Pad1.18x1.45mm_HandSolder, F.Cu at (145.8, 127.0)
- added C2: 5x1uF, Capacitor_THT:C_Rect_L18.0mm_W5.0mm_P15.00mm_FKS3_FKP3, F.Cu at (120.7, 73.5)
- added C3: 5x1uF, Capacitor_THT:C_Rect_L18.0mm_W5.0mm_P15.00mm_FKS3_FKP3, F.Cu at (106.0, 88.5)
- added C4: 10n, Capacitor_THT:C_Rect_L13.0mm_W5.0mm_P10.00mm_FKS3_FKP3_MKS4, F.Cu at (84.1, 59.3)
- added C5: 10n, Capacitor_THT:C_Rect_L13.0mm_W5.0mm_P10.00mm_FKS3_FKP3_MKS4, F.Cu at (89.6, 69.3)
- added C6: 10n, Capacitor_THT:C_Rect_L13.0mm_W5.0mm_P10.00mm_FKS3_FKP3_MKS4, F.Cu at (143.4, 59.7)
- added C7: 10n, Capacitor_THT:C_Rect_L13.0mm_W5.0mm_P10.00mm_FKS3_FKP3_MKS4, F.Cu at (149.0, 69.7)
- added C8: 10u, Capacitor_SMD:C_0805_2012Metric_Pad1.18x1.45mm_HandSolder, F.Cu at (109.6, 134.6)
- added C9: 10u, Capacitor_SMD:C_0805_2012Metric_Pad1.18x1.45mm_HandSolder, F.Cu at (109.6, 137.6)
- added D1: GBJ1008-BP, Snapeda:GBJ1008-BP_DIOB_GBJ1008-BP, F.Cu at (69.5, 103.1)
- added D2: 16V Zener, Diode_SMD:D_0805_2012Metric, F.Cu at (62.9, 33.0)
- added D3: SUF4007, Diode_SMD:D_MELF_Handsoldering, F.Cu at (144.0, 118.5)
- added D4: SUF4007, Diode_SMD:D_MELF_Handsoldering, F.Cu at (127.0, 118.5)
- added D5: 16V Zener, Diode_SMD:D_0805_2012Metric, F.Cu at (62.9, 36.0)
- added D6: SUF4007, Diode_SMD:D_MELF_Handsoldering, F.Cu at (137.4, 131.9)
- added D7: SUF4007, Diode_SMD:D_MELF_Handsoldering, F.Cu at (170.4, 52.1)
- added D8: SUF4007, Diode_SMD:D_MELF_Handsoldering, F.Cu at (170.4, 56.4)
- added J1: Screw_Terminal_01x03, TerminalBlock_4Ucon:TerminalBlock_4Ucon_1x03_P3.50mm_Horizontal, F.Cu at (67.1, 73.3)
- added J2: Screw_Terminal_01x02, TerminalBlock_4Ucon:TerminalBlock_4Ucon_1x02_P3.50mm_Horizontal, F.Cu at (114.5, 50.1)
- added J3: Screw_Terminal_01x02, TerminalBlock_4Ucon:TerminalBlock_4Ucon_1x02_P3.50mm_Horizontal, F.Cu at (156.2, 141.9)
- added L2: AS101, Snapeda:ASM-010_ASM-010, F.Cu at (114.6, 63.8)
- added Q1: Q_NIGBT_GCE, Package_TO_SOT_THT:TO-247-3_Vertical, F.Cu at (77.6, 50.0)
- added Q2: Q_NIGBT_GCE, Package_TO_SOT_THT:TO-247-3_Vertical, F.Cu at (137.6, 50.0)
- added R1: 10R, Resistor_SMD:R_0603_1608Metric_Pad0.98x0.95mm_HandSolder, F.Cu at (138.9, 115.0)
- added R10: 100k, Resistor_THT:R_Axial_DIN0207_L6.3mm_D2.5mm_P7.62mm_Horizontal, F.Cu at (114.6, 92.5)
- added R11: 1k, Resistor_THT:R_Axial_DIN0207_L6.3mm_D2.5mm_P7.62mm_Horizontal, F.Cu at (103.5, 59.7)
- added R2: 10R, Resistor_SMD:R_0603_1608Metric_Pad0.98x0.95mm_HandSolder, F.Cu at (132.7, 115.4)
- added R3: 10R, Resistor_SMD:R_0603_1608Metric_Pad0.98x0.95mm_HandSolder, F.Cu at (138.9, 117.5)
- added R4: 10R, Resistor_SMD:R_0603_1608Metric_Pad0.98x0.95mm_HandSolder, F.Cu at (132.7, 118.1)
- added R5: 10R, Resistor_THT:R_Axial_Power_L25.0mm_W9.0mm_P10.16mm_Vertical, F.Cu at (76.7, 69.0)
- added R6: 10R, Resistor_THT:R_Axial_Power_L25.0mm_W9.0mm_P10.16mm_Vertical, F.Cu at (135.8, 69.4)
- added R7: 10R, Resistor_SMD:R_0603_1608Metric_Pad0.98x0.95mm_HandSolder, F.Cu at (138.9, 120.0)
- added R8: 10R, Resistor_SMD:R_0603_1608Metric_Pad0.98x0.95mm_HandSolder, F.Cu at (132.7, 120.0)
- added R9: 100k, Resistor_THT:R_Axial_DIN0207_L6.3mm_D2.5mm_P7.62mm_Horizontal, F.Cu at (104.7, 92.5)
- added U1: UCC27712D, Snapeda:UCC27712D_SOIC127P599X175-8N, F.Cu at (137.0, 126.5)
- added U2: L78L15_SO8, Package_SO:SOIC-8_3.9x4.9mm_P1.27mm, F.Cu at (158.0, 131.0)
- added U3: ZC323000, Snapeda:ZC323000_MODULE_ZC323000, F.Cu at (92.0, 135.0)
- added U4: HT7533-1-SOT89, Package_TO_SOT_SMD:SOT-89-3, F.Cu at (115.5, 137.1)
- added kibuzzard-65AE80BD: G***, kibuzzard-65AE80BD, F.Cu at (65.1, 91.3)
- added kibuzzard-65AE9F97: G***, kibuzzard-65AE9F97, F.Cu at (114.6, 63.8)
Routing:
- net Net-(D2-A): track 0.00 -> 126.7 mm
- net Net-(Q1-C): track 0.00 -> 115.2 mm
- net Net-(D5-A): track 0.00 -> 87.9 mm
- net Net-(J1-Pin_2): track 0.00 -> 36.5 mm
- net Net-(C2-Pad1): track 0.00 -> 33.7 mm
- net Net-(C6-Pad1): track 0.00 -> 12.9 mm
- net Net-(C4-Pad1): track 0.00 -> 12.7 mm
- net Net-(J2-Pin_1): track 0.00 -> 6.22 mm
- net Net-(C6-Pad2): track 0.00 -> 5.59 mm
- net Net-(C4-Pad2): track 0.00 -> 5.59 mm
- added copper zone on F.Cu, net Net-(C2-Pad1)

Commit message: layout 2nd rev
Parts:
- removed D8: SUF4007, Diode_SMD:D_MELF_Handsoldering
- removed L2: AS101, Snapeda:ASM-010_ASM-010
- removed kibuzzard-65AE9F97: G***, kibuzzard-65AE9F97
- added C10: 220uF, Capacitor_THT:CP_Radial_D22.0mm_P10.00mm_SnapIn, F.Cu at (135.0, 112.5)
- added C11: 220uF, Capacitor_THT:CP_Radial_D22.0mm_P10.00mm_SnapIn, F.Cu at (112.2, 112.5)
- added C15: 220uF, Capacitor_THT:CP_Radial_D22.0mm_P10.00mm_SnapIn, F.Cu at (123.6, 92.7)
- added C16: 4x100nF, Capacitor_SMD:C_0603_1608Metric, F.Cu at (77.9, 76.0)
- added J4: MCSP-Q-08-A-SG-T_R, Samacsys:MCSPQ08ASGTR, F.Cu at (122.7, 139.4)
- added JP1: Solder Jumper, Jumper:SolderJumper-2_P1.3mm_Open_TrianglePad1.0x1.5mm, F.Cu at (96.7, 60.9)
- added JP2: Solder Jumper, Jumper:SolderJumper-2_P1.3mm_Open_TrianglePad1.0x1.5mm, F.Cu at (84.3, 55.1)
- added JP3: Solder Jumper, Jumper:SolderJumper-2_P1.3mm_Open_TrianglePad1.0x1.5mm, F.Cu at (69.3, 57.1)
- added JP4: Solder Jumper, Jumper:SolderJumper-2_P1.3mm_Open_TrianglePad1.0x1.5mm, F.Cu at (74.6, 57.0)
- added JP5: Solder Jumper, Jumper:SolderJumper-2_P1.3mm_Open_TrianglePad1.0x1.5mm, F.Cu at (66.5, 57.1)
- added JP6: Solder Jumper, Jumper:SolderJumper-2_P1.3mm_Open_TrianglePad1.0x1.5mm, F.Cu at (78.1, 78.9)
- added JP7: Solder Jumper, Jumper:SolderJumper-2_P1.3mm_Open_TrianglePad1.0x1.5mm, F.Cu at (78.1, 81.4)
- added JP8: Solder Jumper, Jumper:SolderJumper-2_P1.3mm_Open_TrianglePad1.0x1.5mm, F.Cu at (81.6, 81.4)
- added R12: 1k, Resistor_SMD:R_0603_1608Metric_Pad0.98x0.95mm_HandSolder, F.Cu at (91.2, 131.5)
- added R13: 10k, Resistor_SMD:R_0603_1608Metric_Pad0.98x0.95mm_HandSolder, F.Cu at (88.1, 131.5)
- added R14: 1k, Resistor_SMD:R_0603_1608Metric_Pad0.98x0.95mm_HandSolder, F.Cu at (89.7, 131.5)
- added R15: 1k, Resistor_SMD:R_0603_1608Metric_Pad0.98x0.95mm_HandSolder, F.Cu at (93.3, 126.2)
- added R16: 10R, Resistor_SMD:R_0603_1608Metric_Pad0.98x0.95mm_HandSolder, F.Cu at (73.4, 126.2)
- added R17: 10R, Resistor_SMD:R_0603_1608Metric_Pad0.98x0.95mm_HandSolder, F.Cu at (73.4, 128.0)
- added R18: 1k, Resistor_SMD:R_0603_1608Metric_Pad0.98x0.95mm_HandSolder, F.Cu at (95.2, 131.6)
- added R19: 1k, Resistor_SMD:R_0603_1608Metric_Pad0.98x0.95mm_HandSolder, F.Cu at (96.8, 131.6)
- added RV1: 10k pot, Snapeda:potentiometer, F.Cu at (98.4, 146.5)
- added T1: Gate drive transformer, Transformer_THT:Transformer_Toroid_Tapped_Horizontal_D10.5mm_Amidon-T37, F.Cu at (83.8, 70.9)
- added kibuzzard-65B138E2: G***, kibuzzard-65B138E2, F.Cu at (88.0, 65.1)
- added kibuzzard-65B13903: G***, kibuzzard-65B13903, F.Cu at (87.8, 71.7)
- added kibuzzard-65B13918: G***, kibuzzard-65B13918, F.Cu at (87.8, 60.7)
- C1: value 20uF -> 220uF; footprint Capacitor_THT:CP_Radial_D17.0mm_P7.50mm -> Capacitor_THT:CP_Radial_D22.0mm_P10.00mm_SnapIn
- C12: value 0.1u -> 100nF; footprint Capacitor_SMD:C_0805_2012Metric_Pad1.18x1.45mm_HandSolder -> Capacitor_SMD:C_0603_1608Metric
- C13: value 1u -> 100nF; footprint Capacitor_SMD:C_0805_2012Metric_Pad1.18x1.45mm_HandSolder -> Capacitor_SMD:C_0603_1608Metric
- C14: value 20uF -> 100nF; footprint Capacitor_SMD:C_0805_2012Metric_Pad1.18x1.45mm_HandSolder -> Capacitor_SMD:C_0603_1608Metric
- D2, D5: value 16V Zener -> LED; footprint Diode_SMD:D_0805_2012Metric -> LED_SMD:LED_0805_2012Metric
- D7: value SUF4007 -> LED; footprint Diode_SMD:D_MELF_Handsoldering -> LED_SMD:LED_0805_2012Metric
- R11: footprint Resistor_THT:R_Axial_DIN0207_L6.3mm_D2.5mm_P7.62mm_Horizontal -> Resistor_SMD:R_0603_1608Metric_Pad0.98x0.95mm_HandSolder
- U2: value L78L15_SO8 -> LM317_TO-220; footprint Package_SO:SOIC-8_3.9x4.9mm_P1.27mm -> Package_TO_SOT_THT:TO-220-3_Vertical
- moved D7 110.8 mm to (93.2, 131.6), turned to -90 degrees
- moved D2 97.0 mm to (89.8, 126.2), turned to 180 degrees
- moved D5 96.1 mm to (89.8, 128.3), turned to 180 degrees
- moved kibuzzard-65AE80BD 95.4 mm to (160.5, 93.0)
- moved C13 95.2 mm to (76.4, 76.0), turned to 90 degrees
- moved C12 95.0 mm to (74.9, 76.0), turned to 90 degrees
- moved J1 90.2 mm to (157.0, 80.0), turned to 90 degrees
- moved D6 89.8 mm to (70.4, 72.1)
- moved D3 89.3 mm to (72.6, 64.8)
- moved C14 88.5 mm to (73.4, 76.0), turned to 90 degrees
- moved R7 88.4 mm to (69.6, 65.1), turned to -90 degrees
- moved D1 86.6 mm to (156.0, 98.9), turned to 90 degrees
- moved R8 86.1 mm to (69.6, 61.5), turned to 90 degrees
- moved R3 84.7 mm to (75.4, 61.5), turned to 90 degrees
- moved U1 84.6 mm to (68.7, 76.6)
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Connections:
- C1 pad 2: Net-(D2-A) -> Net-(J2-Pin_1)
- C12 pad 1: +15V -> Net-(JP6-A)
- C12 pad 2: Earth -> Net-(D6-K)
- C13 pad 1: Net-(J3-Pin_2) -> Net-(JP6-A)
- C13 pad 2: Earth -> Net-(D6-K)
- C14 pad 1: Net-(U1-HS) -> Net-(JP6-A)
- C2 pad 1: Net-(C2-Pad1) -> Net-(J2-Pin_1)
- C2 pad 2: Net-(D2-A) -> Bridge_Low
- C3 pad 2: Net-(C2-Pad1) -> Net-(J2-Pin_1)
- C5 pad 2: Net-(D5-A) -> Bridge_Midpoint
- C7 pad 2: Net-(D2-A) -> Bridge_Low
- D1 pad 1: Net-(D2-A) -> Bridge_Low
- D3 pad 2: Net-(D3-A) -> DriverOut_LOW
- D4 pad 2: Net-(D2-K) -> DriverOut_HIGH
- D5 pad 1: Net-(D3-A) -> Net-(D5-K)
- D6 pad 2: +15V -> Net-(D6-A)
- D7 pad 1: +3.3V -> Net-(D7-K)
- D7 pad 2: Current Sense -> +15V
- J2 pad 2: Net-(D5-A) -> Bridge_Midpoint
- Q1 pad 1: Net-(D3-A) -> Net-(JP1-B)
- Q1 pad 3: Net-(D5-A) -> Bridge_Midpoint
- Q2 pad 1: Net-(D2-K) -> Net-(JP2-B)
- Q2 pad 2: Net-(D5-A) -> Bridge_Midpoint
- Q2 pad 3: Net-(D2-A) -> Bridge_Low
- R1 pad 1: GateDrive_HIGH -> Net-(U1-LO)
- R1 pad 2: Net-(D3-A) -> Net-(D3-K)
- R10 pad 1: Net-(C2-Pad1) -> Net-(J2-Pin_1)
- R10 pad 2: Net-(D2-A) -> Bridge_Low
- R11 pad 1: Net-(L2-PadP$2) -> Earth
- R11 pad 2: Current Sense -> Net-(D5-K)
- R2 pad 1: GateDrive_LOW -> Net-(U1-LO)
- R2 pad 2: Net-(D4-K) -> Net-(D3-K)
- R3 pad 1: GateDrive_HIGH -> Net-(U1-LO)
- R3 pad 2: Net-(D3-K) -> DriverOut_LOW
- R4 pad 1: GateDrive_LOW -> Net-(U1-HO)
- R4 pad 2: Net-(D2-K) -> Net-(D4-K)
- R6 pad 2: Net-(D5-A) -> Bridge_Midpoint
- R7 pad 1: GateDrive_HIGH -> Net-(U1-HO)
- R7 pad 2: Net-(D3-K) -> Net-(D4-K)
- R8 pad 1: GateDrive_LOW -> Net-(U1-HO)
- R8 pad 2: Net-(D4-K) -> DriverOut_HIGH
- R9 pad 2: Net-(C2-Pad1) -> Net-(J2-Pin_1)
- U1 pad 1: PWM_LOW -> Net-(U1-LL)
- U1 pad 2: PWM_HIGH -> Net-(U1-HL)
- U1 pad 3: +15V -> Net-(D6-A)
- U1 pad 5: GateDrive_LOW -> Net-(U1-LO)
- U1 pad 6: Net-(U1-HS) -> Net-(JP6-A)
- U1 pad 7: GateDrive_HIGH -> Net-(U1-HO)
- U2 pad 1: +15V -> Net-(U2-ADJ)
- U2 pad 2: Earth -> +15V
- U2 pad 3: Earth -> Net-(J3-Pin_2)
- U3 pad 10: unconnected-(U3-A5-Pad10) -> Net-(J4-CLX)
- U3 pad 11: unconnected-(U3-A6-Pad11) -> Net-(J4-DAT0)
- U3 pad 12: unconnected-(U3-A7-Pad12) -> Net-(J4-CMD)
- U3 pad 13: PWM_LOW -> PWM_HIGH
- U3 pad 14: PWM_HIGH -> PWM_LOW
- U3 pad 15: unconnected-(U3-B10-Pad15) -> Net-(D2-A)
- U3 pad 16: unconnected-(U3-B11-Pad16) -> Net-(D5-A)
- U3 pad 6: Current Sense -> Net-(U3-A1)
- U3 pad 9: unconnected-(U3-A4-Pad9) -> Net-(J4-CD/DAT3)
Routing:
- net Net-(Q1-C): track 115.2 -> 0.00 mm
- net Net-(D2-A): track 126.7 -> 22.8 mm
- net Net-(U3-A1): track 0.00 -> 84.0 mm, vias 0 -> 1
- net Net-(JP1-B): track 0.00 -> 68.9 mm
- net +3.3V: track 0.00 -> 68.3 mm
- net Net-(U1-LL): track 0.00 -> 66.1 mm
- net Net-(JP2-B): track 0.00 -> 65.0 mm, vias 0 -> 1
- net Net-(D5-A): track 87.9 -> 23.0 mm
- net Net-(U1-HL): track 0.00 -> 59.3 mm
- net Earth: track 0.00 -> 44.1 mm, vias 0 -> 3
- net Net-(J1-Pin_2): track 36.5 -> 0.00 mm
- net Net-(C2-Pad1): track 33.7 -> 0.00 mm
- net DriverOut_LOW: track 0.00 -> 27.4 mm
- net Bridge_Low: track 0.00 -> 26.1 mm, vias 0 -> 1
- net +15V: track 0.00 -> 25.3 mm, vias 0 -> 1
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- added copper zone on F.Cu, net Earth
- removed copper zone on F.Cu, net Net-(C2-Pad1)

Commit message: routing, power traces
Parts:
- moved C2 3.48 mm to (133.0, 72.9)
- moved J2 1.27 mm to (157.4, 58.1)
Routing:
- net Bridge_Low: track 26.1 -> 90.6 mm
- net Net-(J4-CD/DAT3): track 0.00 -> 63.5 mm
- net Bridge_Midpoint: track 14.8 -> 78.0 mm, vias 0 -> 6
- net Net-(J4-CMD): track 0.00 -> 58.8 mm, vias 0 -> 2
- net Net-(J4-CLX): track 0.00 -> 58.5 mm
- net Net-(J4-DAT0): track 0.00 -> 57.6 mm
- net Earth: track 44.1 -> 98.9 mm, vias 3 -> 7
- net +3.3V: track 68.3 -> 92.0 mm
- net Net-(J1-Pin_2): track 0.00 -> 21.6 mm
- net Net-(Q1-C): track 0.00 -> 15.9 mm, vias 0 -> 14
- net Net-(C6-Pad1): track 0.00 -> 12.9 mm
- net Net-(C4-Pad1): track 0.00 -> 12.7 mm
- net Net-(C6-Pad2): track 0.00 -> 5.59 mm
- net Net-(C4-Pad2): track 0.00 -> 5.59 mm
- net Net-(JP3-B): track 24.8 -> 24.1 mm
- added copper zone on B.Cu, net Bridge_Low
- added copper zone on F.Cu, net Bridge_Low
- added copper zone on B.Cu, net Bridge_Midpoint
- added copper zone on F.Cu, net Bridge_Midpoint
- added copper zone on B.Cu, net Net-(J2-Pin_1)
- added copper zone on F.Cu, net Net-(J2-Pin_1)
- added copper zone on B.Cu, net Net-(Q1-C)
- added copper zone on F.Cu, net Net-(Q1-C)
