File: TeslaCoil.kicad_pcb (KiCad board)
At the start: 2 copper layers, 100 x 101 mm, 68 parts, among them J1 Screw_Terminal_01x03, J2 Screw_Terminal_01x02, J3 Screw_Terminal_01x02, J4 MCSP-Q-08-A-SG-T_R, Q1 Q_NIGBT_GCE, Q2 Q_NIGBT_GCE, T1 Gate drive transformer, U1 UCC27712D, U2 LM317_TO-220, U3 ZC323000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

Commit message: final v1
Parts:
- removed kibuzzard-65AE80BD: G***, kibuzzard-65AE80BD
- added REF**: MountingHole_3.2mm_M3_Pad_Via, MountingHole:MountingHole_3.2mm_M3_Pad_Via, F.Cu at (159.4, 49.5)
- added SW1: SW_SPST, Snapeda:Rocker switch, F.Cu at (156.7, 131.3)
- added kibuzzard-65B38B8A: G***, kibuzzard-65B38B8A, F.Cu at (160.0, 77.0)
- added kibuzzard-65B38BA7: G***, kibuzzard-65B38BA7, F.Cu at (91.7, 145.5)
- added kibuzzard-65B38BC8: G***, kibuzzard-65B38BC8, F.Cu at (160.0, 57.7)
- T1: value Gate drive transformer -> GDT
- moved J2 1.36 mm to (157.0, 59.4)
Connections:
- J1 pad 1: unconnected-(J1-Pin_1-Pad1) -> Earth
- REF** pad 1: (no net) -> Earth (x2)
Routing:
- net Earth: track 99.3 -> 274.8 mm, vias 7 -> 8
- net Net-(J1-Pin_3): track 0.00 -> 65.9 mm
- net Net-(SW1-B): track 0.00 -> 30.9 mm
Other:
- board text added: "Tesla coil inverter v.1 Degesz 2024"
- board text added: "sus"

Commit message: production v1
Other:
- board text added: "JLCJLCJLCJLC"
Changed lines of the file:
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@@
     (property "ki_keywords" "switch lever")
     (attr through_hole)
-    (fp_text reference "SW1" (at -0.302 -2.54 90 unlocked) (layer "F.SilkS")
+    (fp_text reference "SW1" (at -0.302 -2.54 90 unlocked) (layer "F.SilkS") hide
         (effects (font (size 1 1) (thickness 0.15)))
     )
@@
     (fp_line (start 2.6 1.3) (end 2.6 -1.3)
       (stroke (width 0.1) (type solid)) (layer "F.Fab"))
-    (pad "1" smd roundrect (at -3.4 0 90) (size 3.5 2.7) (layers "F.Cu" "F.Paste" "F.Mask") (roundrect_rratio 0.0925925926)
+    (pad "1" smd roundrect (at -3.4 0 90) (size 3.5 2.7) (layers "F.Cu" "F.Paste" "F.Mask") (roundrect_rratio 0.09259259259)
       (net 14 "Net-(D4-K)") (pinfunction "K") (pintype "passive"))
-    (pad "2" smd roundrect (at 3.4 0 90) (size 3.5 2.7) (layers "F.Cu" "F.Paste" "F.Mask") (roundrect_rratio 0.0925925926)
+    (pad "2" smd roundrect (at 3.4 0 90) (size 3.5 2.7) (layers "F.Cu" "F.Paste" "F.Mask") (roundrect_rratio 0.09259259259)
       (net 54 "DriverOut_HIGH") (pinfunction "A") (pintype "passive"))
     (model "${KICAD6_3DMODEL_DIR}/Diode_SMD.3dshapes/D_MELF.wrl"
@@
     (fp_line (start 1 0.625) (end -1 0.625)
       (stroke (width 0.1) (type solid)) (layer "F.Fab"))
-    (pad "1" smd roundrect (at -1.0375 0 270) (size 1.175 1.45) (layers "F.Cu" "F.Paste" "F.Mask") (roundrect_rratio 0.212766)
+    (pad "1" smd roundrect (at -1.0375 0 270) (size 1.175 1.45) (layers "F.Cu" "F.Paste" "F.Mask") (roundrect_rratio 0.2127659574)
       (net 7 "+15V") (pintype "passive"))
-    (pad "2" smd roundrect (at 1.0375 0 270) (size 1.175 1.45) (layers "F.Cu" "F.Paste" "F.Mask") (roundrect_rratio 0.212766)
+    (pad "2" smd roundrect (at 1.0375 0 270) (size 1.175 1.45) (layers "F.Cu" "F.Paste" "F.Mask") (roundrect_rratio 0.2127659574)
       (net 50 "Earth") (pintype "passive"))
     (model "${KICAD6_3DMODEL_DIR}/Capacitor_SMD.3dshapes/C_0805_2012Metric.wrl"
@@
     (fp_line (start 2.6 1.3) (end 2.6 -1.3)
       (stroke (width 0.1) (type solid)) (layer "F.Fab"))
-    (pad "1" smd roundrect (at -3.4 0 90) (size 3.5 2.7) (layers "F.Cu" "F.Paste" "F.Mask") (roundrect_rratio 0.0925925926)
+    (pad "1" smd roundrect (at -3.4 0 90) (size 3.5 2.7) (layers "F.Cu" "F.Paste" "F.Mask") (roundrect_rratio 0.09259259259)
       (net 13 "Net-(D3-K)") (pinfunction "K") (pintype "passive"))
-    (pad "2" smd roundrect (at 3.4 0 90) (size 3.5 2.7) (layers "F.Cu" "F.Paste" "F.Mask") (roundrect_rratio 0.0925925926)
+    (pad "2" smd roundrect (at 3.4 0 90) (size 3.5 2.7) (layers "F.Cu" "F.Paste" "F.Mask") (roundrect_rratio 0.09259259259)
       (net 53 "DriverOut_LOW") (pinfunction "A") (pintype "passive"))
     (model "${KICAD6_3DMODEL_DIR}/Diode_SMD.3dshapes/D_MELF.wrl"
@@
     (fp_line (start 1 0.625) (end -1 0.625)
       (stroke (width 0.1) (type solid)) (layer "F.Fab"))
-    (pad "1" smd roundrect (at -1.0375 0 270) (size 1.175 1.45) (layers "F.Cu" "F.Paste" "F.Mask") (roundrect_rratio 0.212766)
+    (pad "1" smd roundrect (at -1.0375 0 270) (size 1.175 1.45) (layers "F.Cu" "F.Paste" "F.Mask") (roundrect_rratio 0.2127659574)
       (net 8 "+3.3V") (pintype "passive"))
-    (pad "2" smd roundrect (at 1.0375 0 270) (size 1.175 1.45) (layers "F.Cu" "F.Paste" "F.Mask") (roundrect_rratio 0.212766)
+    (pad "2" smd roundrect (at 1.0375 0 270) (size 1.175 1.45) (layers "F.Cu" "F.Paste" "F.Mask") (roundrect_rratio 0.2127659574)
       (net 50 "Earth") (pintype "passive"))
     (model "${KICAD6_3DMODEL_DIR}/Capacitor_SMD.3dshapes/C_0805_2012Metric.wrl"
@@
     (fp_line (start 2.6 1.3) (end 2.6 -1.3)
       (stroke (width 0.1) (type solid)) (layer "F.Fab"))
-    (pad "1" smd roundrect (at -3.4 0 180) (size 3.5 2.7) (layers "F.Cu" "F.Paste" "F.Mask") (roundrect_rratio 0.0925925926)
+    (pad "1" smd roundrect (at -3.4 0 180) (size 3.5 2.7) (layers "F.Cu" "F.Paste" "F.Mask") (roundrect_rratio 0.09259259259)
       (net 10 "Net-(D6-K)") (pinfunction "K") (pintype "passive"))
-    (pad "2" smd roundrect (at 3.4 0 180) (size 3.5 2.7) (layers "F.Cu" "F.Paste" "F.Mask") (roundrect_rratio 0.0925925926)
+    (pad "2" smd roundrect (at 3.4 0 180) (size 3.5 2.7) (layers "F.Cu" "F.Paste" "F.Mask") (roundrect_rratio 0.09259259259)
       (net 57 "Net-(D6-A)") (pinfunction "A") (pintype "passive"))
     (model "${KICAD6_3DMODEL_DIR}/Diode_SMD.3dshapes/D_MELF.wrl"
@@
     (effects (font (size 0.5 0.5) (thickness 0.1) bold) (justify left bottom))
   )
+  (gr_text "JLCJLCJLCJLC" (at 69.596 100.838 270) (layer "F.SilkS")
+    (effects (font (size 1 1) (thickness 0.1)) (justify left bottom))
+  )
   (gr_text_box "Heatsink\n"
