File: TeslaCoil.stretch_bkup.kicad_pcb (KiCad board)
At the start: 2 copper layers, 100 x 101 mm, 68 parts, among them J1 Screw_Terminal_01x03, J2 Screw_Terminal_01x02, J3 Screw_Terminal_01x02, J4 MCSP-Q-08-A-SG-T_R, Q1 Q_NIGBT_GCE, Q2 Q_NIGBT_GCE, T1 Gate drive transformer, U1 UCC27712D, U2 LM317_TO-220, U3 ZC323000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

Commit message: amogus
Parts:
- removed REF** (x2): MountingHole_3.2mm_M3_Pad_Via, MountingHole:MountingHole_3.2mm_M3_Pad_Via
Routing:
- net +3.3V: track 145.2 -> 92.0 mm, vias 2 -> 0
